File: vfo/vfo.sch (KiCad schematic (older format))
At the start: 20 parts, among them J1 CV In Jack, J2 Sawtooth Output, J3 Triangle Output, J5 Conn_01x06, J6 Bus 16 pin, U1 TL072, U2 AS3340

Commit message: Reworked for 24mm wide
Parts:
- removed J5: Conn_01x06, Connector_PinHeader_2.54mm:PinHeader_1x06_P2.54mm_Vertical, symbol Connector_Generic:Conn_01x06
- removed J6: Bus 16 pin, Connector_PinHeader_2.54mm:PinHeader_2x08_P2.54mm_Vertical, symbol Connector_Generic:Conn_02x08_Odd_Even
- added J4: Conn_02x05_Odd_Even, Connector_PinHeader_2.54mm:PinHeader_2x05_P2.54mm_Vertical, symbol Connector_Generic:Conn_02x05_Odd_Even
- added J5: Conn_01x08, Connector_PinHeader_2.54mm:PinHeader_1x08_P2.54mm_Vertical, symbol Connector_Generic:Conn_01x08
- J1: value CV In Jack -> CVIN
- J2: value Sawtooth Output -> SAW
- J3: value Triangle Output -> TRI
- RV2: footprint Potentiometer_THT:Potentiometer_Bourns_3386F_Vertical -> Potentiometer_SMD:Potentiometer_Bourns_3314J_Vertical
Connections:
- net labels removed: +5V, CV_BUS, GATE_BUS
- wire segments 59 -> 55
Changed lines of the file:
@@
 F 0 "RV2" V 6600 1100 50  0000 C CNN
 F 1 "10K" V 6750 1100 50  0000 C CNN
-F 2 "Potentiometer_THT:Potentiometer_Bourns_3386F_Vertical" H 6750 1100 50  0001 C CNN
+F 2 "Potentiometer_SMD:Potentiometer_Bourns_3314J_Vertical" H 6750 1100 50  0001 C CNN
 F 3 "~" H 6750 1100 50  0001 C CNN
 	1    6750 1100
@@
 Wire Notes Line
 	800  3250 11150 3250
-$Comp
-L Connector_Generic:Conn_01x06 J5
-U 1 1 5B6FAFE0
-P 8300 3600
-F 0 "J5" H 8380 3592 50  0000 L CNN
-F 1 "Conn_01x06" H 8380 3501 50  0000 L CNN
-F 2 "Connector_PinHeader_2.54mm:PinHeader_1x06_P2.54mm_Vertical" H 8300 3600 50  0001 C CNN
-F 3 "~" H 8300 3600 50  0001 C CNN
-	1    8300 3600
-	1    0    0    -1
-$EndComp
 Wire Wire Line
 	8100 3400 7750 3400
@@
 L power:GND #PWR0123
 U 1 1 5B7035F9
-P 8100 3900
-F 0 "#PWR0123" H 8100 3650 50  0001 C CNN
-F 1 "GND" H 8105 3727 50  0000 C CNN
-F 2 "" H 8100 3900 50  0001 C CNN
-F 3 "" H 8100 3900 50  0001 C CNN
-	1    8100 3900
-	1    0    0    -1
+P 8100 4000
+F 0 "#PWR0123" H 8100 3750 50  0001 C CNN
+F 1 "GND" V 8100 3800 50  0000 C CNN
+F 2 "" H 8100 4000 50  0001 C CNN
+F 3 "" H 8100 4000 50  0001 C CNN
+	1    8100 4000
+	0    1    1    0
 $EndComp
 $Comp
@@
 P 1800 1150
 F 0 "J1" H 1720 825 50  0000 C CNN
-F 1 "CV In Jack" H 1720 916 50  0000 C CNN
+F 1 "CVIN" H 1720 916 50  0000 C CNN
 F 2 "Connector_PinHeader_2.54mm:PinHeader_1x02_P2.54mm_Vertical" H 1800 1150 50  0001 C CNN
 F 3 "~" H 1800 1150 50  0001 C CNN
@@
 P 1800 2150
 F 0 "J2" H 1720 1825 50  0000 C CNN
-F 1 "Sawtooth Output" H 1720 1916 50  0000 C CNN
+F 1 "SAW" H 1720 1916 50  0000 C CNN
 F 2 "Connector_PinHeader_2.54mm:PinHeader_1x02_P2.54mm_Vertical" H 1800 2150 50  0001 C CNN
 F 3 "~" H 1800 2150 50  0001 C CNN
@@
 P 1800 2850
 F 0 "J3" H 1720 2525 50  0000 C CNN
-F 1 "Triangle Output" H 1720 2616 50  0000 C CNN
+F 1 "TRI" H 1720 2616 50  0000 C CNN
 F 2 "Connector_PinHeader_2.54mm:PinHeader_1x02_P2.54mm_Vertical" H 1800 2850 50  0001 C CNN
 F 3 "~" H 1800 2850 50  0001 C CNN
@@
 Wire Notes Line
 	8950 3250 8950 4300
-Wire Notes Line
-	7550 3250 7550 4300
-Text Notes 9900 4450 0    50   ~ 0
+Text Notes 9900 4200 0    50   ~ 0
 Power Bus
-Text Notes 7750 4250 0    50   ~ 0
+Text Notes 7750 4550 0    50   ~ 0
 Disconnected Pin Breakout
 Text Notes 6650 3150 0    50   ~ 0
@@
 Tuning
 $Comp
-L Connector_Generic:Conn_02x08_Odd_Even J6
-U 1 1 5B6F6B88
-P 10050 3850
-F 0 "J6" H 10100 4367 50  0000 C CNN
-F 1 "Bus 16 pin" H 10100 4276 50  0000 C CNN
-F 2 "Connector_PinHeader_2.54mm:PinHeader_2x08_P2.54mm_Vertical" H 10050 3850 50  0001 C CNN
-F 3 "~" H 10050 3850 50  0001 C CNN
-	1    10050 3850
-	1    0    0    -1
-$EndComp
-Wire Wire Line
-	10350 3550 10750 3550
-Wire Wire Line
-	9850 3550 9450 3550
-Wire Wire Line
-	10350 3650 10750 3650
-$Comp
 L power:GND #PWR0124
 U 1 1 5B6FAF73
-P 10350 3950
-F 0 "#PWR0124" H 10350 3700 50  0001 C CNN
-F 1 "GND" V 10355 3822 50  0000 R CNN
-F 2 "" H 10350 3950 50  0001 C CNN
-F 3 "" H 10350 3950 50  0001 C CNN
-	1    10350 3950
+P 10350 3700
+F 0 "#PWR0124" H 10350 3450 50  0001 C CNN
+F 1 "GND" V 10350 3550 50  0000 R CNN
+F 2 "" H 10350 3700 50  0001 C CNN
+F 3 "" H 10350 3700 50  0001 C CNN
+	1    10350 3700
 	0    -1   -1   0
 $EndComp
@@
 L power:GND #PWR0127
 U 1 1 5B6FAF79
-P 10350 4050
-F 0 "#PWR0127" H 10350 3800 50  0001 C CNN
-F 1 "GND" V 10355 3922 50  0000 R CNN
-F 2 "" H 10350 4050 50  0001 C CNN
-F 3 "" H 10350 4050 50  0001 C CNN
-	1    10350 4050
+P 10350 3800
+F 0 "#PWR0127" H 10350 3550 50  0001 C CNN
+F 1 "GND" V 10350 3650 50  0000 R CNN
+F 2 "" H 10350 3800 50  0001 C CNN
+F 3 "" H 10350 3800 50  0001 C CNN
+	1    10350 3800
 	0    -1   -1   0
 $EndComp
@@
 L power:GND #PWR0128
 U 1 1 5B6FAF7F
-P 10350 4150
-F 0 "#PWR0128" H 10350 3900 50  0001 C CNN
-F 1 "GND" V 10355 4022 50  0000 R CNN
-F 2 "" H 10350 4150 50  0001 C CNN
-F 3 "" H 10350 4150 50  0001 C CNN
-	1    10350 4150
+P 10350 3900
+F 0 "#PWR0128" H 10350 3650 50  0001 C CNN
+F 1 "GND" V 10350 3750 50  0000 R CNN
+F 2 "" H 10350 3900 50  0001 C CNN
+F 3 "" H 10350 3900 50  0001 C CNN
+	1    10350 3900
 	0    -1   -1   0
 $EndComp
@@
 L power:+12V #PWR0130
 U 1 1 5B6FAF85
-P 10350 3850
-F 0 "#PWR0130" H 10350 3700 50  0001 C CNN
-F 1 "+12V" V 10365 3978 50  0000 L CNN
-F 2 "" H 10350 3850 50  0001 C CNN
-F 3 "" H 10350 3850 50  0001 C CNN
-	1    10350 3850
+P 10350 3600
+F 0 "#PWR0130" H 10350 3450 50  0001 C CNN
+F 1 "+12V" V 10350 3750 50  0000 L CNN
+F 2 "" H 10350 3600 50  0001 C CNN
+F 3 "" H 10350 3600 50  0001 C CNN
+	1    10350 3600
 	0    1    1    0
 $EndComp
@@
 L power:-12V #PWR0131
 U 1 1 5B6FAF8B
-P 10350 4250
-F 0 "#PWR0131" H 10350 4350 50  0001 C CNN
-F 1 "-12V" V 10365 4378 50  0000 L CNN
-F 2 "" H 10350 4250 50  0001 C CNN
-F 3 "" H 10350 4250 50  0001 C CNN
-	1    10350 4250
+P 10350 4000
+F 0 "#PWR0131" H 10350 4100 50  0001 C CNN
+F 1 "-12V" V 10350 4150 50  0000 L CNN
+F 2 "" H 10350 4000 50  0001 C CNN
+F 3 "" H 10350 4000 50  0001 C CNN
+	1    10350 4000
 	0    1    1    0
 $EndComp
@@
 L power:GND #PWR0132
 U 1 1 5B6FC18B
-P 9850 3950
-F 0 "#PWR0132" H 9850 3700 50  0001 C CNN
-F 1 "GND" V 9855 3822 50  0000 R CNN
-F 2 "" H 9850 3950 50  0001 C CNN
-F 3 "" H 9850 3950 50  0001 C CNN
-	1    9850 3950
+P 9850 3700
+F 0 "#PWR0132" H 9850 3450 50  0001 C CNN
+F 1 "GND" V 9850 3550 50  0000 R CNN
+F 2 "" H 9850 3700 50  0001 C CNN
+F 3 "" H 9850 3700 50  0001 C CNN
+	1    9850 3700
 	0    1    1    0
 $EndComp
@@
 L power:GND #PWR0133
 U 1 1 5B6FC191
-P 9850 4050
-F 0 "#PWR0133" H 9850 3800 50  0001 C CNN
-F 1 "GND" V 9855 3922 50  0000 R CNN
-F 2 "" H 9850 4050 50  0001 C CNN
-F 3 "" H 9850 4050 50  0001 C CNN
-	1    9850 4050
+P 9850 3800
+F 0 "#PWR0133" H 9850 3550 50  0001 C CNN
+F 1 "GND" V 9850 3650 50  0000 R CNN
+F 2 "" H 9850 3800 50  0001 C CNN
+F 3 "" H 9850 3800 50  0001 C CNN
+	1    9850 3800
 	0    1    1    0
 $EndComp
@@
 L power:GND #PWR0134
 U 1 1 5B6FC197
-P 9850 4150
-F 0 "#PWR0134" H 9850 3900 50  0001 C CNN
-F 1 "GND" V 9855 4022 50  0000 R CNN
-F 2 "" H 9850 4150 50  0001 C CNN
-F 3 "" H 9850 4150 50  0001 C CNN
-	1    9850 4150
+P 9850 3900
+F 0 "#PWR0134" H 9850 3650 50  0001 C CNN
+F 1 "GND" V 9850 3750 50  0000 R CNN
+F 2 "" H 9850 3900 50  0001 C CNN
+F 3 "" H 9850 3900 50  0001 C CNN
+	1    9850 3900
 	0    1    1    0
 $EndComp
@@
 L power:+12V #PWR0135
 U 1 1 5B6FC19D
-P 9850 3850
-F 0 "#PWR0135" H 9850 3700 50  0001 C CNN
-F 1 "+12V" V 9865 3978 50  0000 L CNN
-F 2 "" H 9850 3850 50  0001 C CNN
-F 3 "" H 9850 3850 50  0001 C CNN
-	1    9850 3850
+P 9850 3600
+F 0 "#PWR0135" H 9850 3450 50  0001 C CNN
+F 1 "+12V" V 9850 3750 50  0000 L CNN
+F 2 "" H 9850 3600 50  0001 C CNN
+F 3 "" H 9850 3600 50  0001 C CNN
+	1    9850 3600
 	0    -1   -1   0
 $EndComp
@@
 L power:-12V #PWR0136
 U 1 1 5B6FC1A3
-P 9850 4250
-F 0 "#PWR0136" H 9850 4350 50  0001 C CNN
-F 1 "-12V" V 9865 4378 50  0000 L CNN
-F 2 "" H 9850 4250 50  0001 C CNN
-F 3 "" H 9850 4250 50  0001 C CNN
-	1    9850 4250
-	0    -1   -1   0
-$EndComp
-Wire Wire Line
-	9850 3650 9450 3650
-Text Label 9450 3550 0    50   ~ 0
-GATE_BUS
-Text Label 9450 3650 0    50   ~ 0
-CV_BUS
-$Comp
-L power:+5V #PWR0137
-U 1 1 5B6FF8A9
-P 9850 3750
-F 0 "#PWR0137" H 9850 3600 50  0001 C CNN
-F 1 "+5V" V 9865 3878 50  0000 L CNN
-F 2 "" H 9850 3750 50  0001 C CNN
-F 3 "" H 9850 3750 50  0001 C CNN
-	1    9850 3750
-	0    -1   -1   0
-$EndComp
-$Comp
-L power:+5V #PWR0138
-U 1 1 5B6FF96C
-P 10350 3750
-F 0 "#PWR0138" H 10350 3600 50  0001 C CNN
-F 1 "+5V" V 10365 3878 50  0000 L CNN
-F 2 "" H 10350 3750 50  0001 C CNN
-F 3 "" H 10350 3750 50  0001 C CNN
-	1    10350 3750
-	0    1    1    0
-$EndComp
-Text Label 10750 3650 2    50   ~ 0
-CV_BUS
-Text Label 10750 3550 2    50   ~ 0
-GATE_BUS
+P 9850 4000
+F 0 "#PWR0136" H 9850 4100 50  0001 C CNN
+F 1 "-12V" V 9850 4150 50  0000 L CNN
+F 2 "" H 9850 4000 50  0001 C CNN
+F 3 "" H 9850 4000 50  0001 C CNN
+	1    9850 4000
+	0    -1   -1   0
+$EndComp
+$Comp
+L Connector_Generic:Conn_02x05_Odd_Even J4
+U 1 1 5B70CB01
+P 10050 3800
+F 0 "J4" H 10100 4217 50  0000 C CNN
+F 1 "Conn_02x05_Odd_Even" H 10100 4126 50  0000 C CNN
+F 2 "Connector_PinHeader_2.54mm:PinHeader_2x05_P2.54mm_Vertical" H 10050 3800 50  0001 C CNN
+F 3 "~" H 10050 3800 50  0001 C CNN
+	1    10050 3800
+	1    0    0    -1
+$EndComp
+Wire Notes Line
+	11200 4300 7550 4300
+Wire Notes Line
+	7550 3250 7550 4300
+$Comp
+L Connector_Generic:Conn_01x08 J5
+U 1 1 5B7128F2
+P 8300 3700
+F 0 "J5" H 8380 3692 50  0000 L CNN
+F 1 "Conn_01x08" H 8380 3601 50  0000 L CNN
+F 2 "Connector_PinHeader_2.54mm:PinHeader_1x08_P2.54mm_Vertical" H 8300 3700 50  0001 C CNN
+F 3 "~" H 8300 3700 50  0001 C CNN
+	1    8300 3700
+	1    0    0    -1
+$EndComp
+$Comp
+L power:-12V #PWR0102
+U 1 1 5B7148FB
+P 8100 4100
+F 0 "#PWR0102" H 8100 4200 50  0001 C CNN
+F 1 "-12V" V 8100 4250 50  0000 L CNN
+F 2 "" H 8100 4100 50  0001 C CNN
+F 3 "" H 8100 4100 50  0001 C CNN
+	1    8100 4100
+	0    -1   -1   0
+$EndComp
+$Comp
+L power:+12V #PWR0103
+U 1 1 5B714A88
+P 8100 3900
+F 0 "#PWR0103" H 8100 3750 50  0001 C CNN
+F 1 "+12V" V 8100 4050 50  0000 L CNN
+F 2 "" H 8100 3900 50  0001 C CNN
+F 3 "" H 8100 3900 50  0001 C CNN
+	1    8100 3900
+	0    -1   -1   0
+$EndComp
 $EndSCHEMATC

Commit message: Update for 19mm width
Parts:
- removed J5: Conn_01x08, Connector_PinHeader_2.54mm:PinHeader_1x08_P2.54mm_Vertical, symbol Connector_Generic:Conn_01x08
- added J5: Conn_01x06, Connector_PinHeader_2.54mm:PinHeader_1x06_P2.54mm_Vertical, symbol Connector_Generic:Conn_01x06
Changed lines of the file:
@@
 VSSI
-$Comp
-L power:GND #PWR0123
-U 1 1 5B7035F9
-P 8100 4000
-F 0 "#PWR0123" H 8100 3750 50  0001 C CNN
-F 1 "GND" V 8100 3800 50  0000 C CNN
-F 2 "" H 8100 4000 50  0001 C CNN
-F 3 "" H 8100 4000 50  0001 C CNN
-	1    8100 4000
-	0    1    1    0
-$EndComp
 $Comp
 L power:-12V #PWR0107
@@
 	7550 3250 7550 4300
 $Comp
-L Connector_Generic:Conn_01x08 J5
-U 1 1 5B7128F2
-P 8300 3700
-F 0 "J5" H 8380 3692 50  0000 L CNN
-F 1 "Conn_01x08" H 8380 3601 50  0000 L CNN
-F 2 "Connector_PinHeader_2.54mm:PinHeader_1x08_P2.54mm_Vertical" H 8300 3700 50  0001 C CNN
-F 3 "~" H 8300 3700 50  0001 C CNN
-	1    8300 3700
-	1    0    0    -1
-$EndComp
-$Comp
 L power:-12V #PWR0102
 U 1 1 5B7148FB
-P 8100 4100
-F 0 "#PWR0102" H 8100 4200 50  0001 C CNN
-F 1 "-12V" V 8100 4250 50  0000 L CNN
-F 2 "" H 8100 4100 50  0001 C CNN
-F 3 "" H 8100 4100 50  0001 C CNN
-	1    8100 4100
-	0    -1   -1   0
-$EndComp
-$Comp
-L power:+12V #PWR0103
-U 1 1 5B714A88
 P 8100 3900
-F 0 "#PWR0103" H 8100 3750 50  0001 C CNN
-F 1 "+12V" V 8100 4050 50  0000 L CNN
+F 0 "#PWR0102" H 8100 4000 50  0001 C CNN
+F 1 "-12V" V 8100 4050 50  0000 L CNN
 F 2 "" H 8100 3900 50  0001 C CNN
 F 3 "" H 8100 3900 50  0001 C CNN
@@
 	0    -1   -1   0
 $EndComp
+$Comp
+L Connector_Generic:Conn_01x06 J5
+U 1 1 5B716C3B
+P 8300 3600
+F 0 "J5" H 8380 3592 50  0000 L CNN
+F 1 "Conn_01x06" H 8380 3501 50  0000 L CNN
+F 2 "Connector_PinHeader_2.54mm:PinHeader_1x06_P2.54mm_Vertical" H 8300 3600 50  0001 C CNN
+F 3 "~" H 8300 3600 50  0001 C CNN
+	1    8300 3600
+	1    0    0    -1
+$EndComp
 $EndSCHEMATC

Commit message: Add BOM details
Parts:
- C1, C2: MFR (none) -> -; MPN (none) -> CC0805MKX7RYBB103; SPN (none) -> -; SPR (none) -> -; SPURL (none) -> -
- C3: MFR (none) -> -; MPN (none) -> CC0805KRX7RABB102; SPN (none) -> -; SPR (none) -> -; SPURL (none) -> -
- J1, J2, J3, J4, J5, RV1: MFR (none) -> -; MPN (none) -> -; SPN (none) -> -; SPR (none) -> -; SPURL (none) -> -
- R1: MFR (none) -> -; MPN (none) -> RC0805FR-07100KL; SPN (none) -> -; SPR (none) -> -; SPURL (none) -> -
- R2, R7: MFR (none) -> -; MPN (none) -> RC0805FR-07470RL; SPN (none) -> -; SPR (none) -> -; SPURL (none) -> -
- R3: MFR (none) -> -; MPN (none) -> RC0805FR-0724KL; SPN (none) -> -; SPR (none) -> -; SPURL (none) -> -
- R4: MFR (none) -> -; MPN (none) -> RC0805FR-075K6L; SPN (none) -> -; SPR (none) -> -; SPURL (none) -> -
- R5: MFR (none) -> Yageo; MPN (none) -> RC0805FR-071K82L; SPN (none) -> -; SPR (none) -> -; SPURL (none) -> -
- R6: MFR (none) -> -; MPN (none) -> RC0805FR-07820RL; SPN (none) -> -; SPR (none) -> -; SPURL (none) -> -
- R8: MFR (none) -> Yageo; MPN (none) -> RC0805FR-071M5L; SPN (none) -> -; SPR (none) -> -; SPURL (none) -> -
- RV2: MFR (none) -> Bourns; MPN (none) -> ‎3314J-1-103E; SPN (none) -> -; SPR (none) -> -; SPURL (none) -> -
- U1: MFR (none) -> -; MPN (none) -> ‎TL072CDR; SPN (none) -> -; SPR (none) -> -; SPURL (none) -> -
- U2: MFR (none) -> -; MPN (none) -> AS3340; SPN (none) -> -; SPR (none) -> -; SPURL (none) -> -

Commit message: Fix 400R R2 resistor
Parts:
- R2: value 470K -> 470R
Changed lines of the file:
@@
 P 7000 2600
 F 0 "R2" V 6900 2600 50  0000 C CNN
-F 1 "470K" V 7000 2600 50  0000 C CNN
+F 1 "470R" V 7000 2600 50  0000 C CNN
 F 2 "Resistor_SMD:R_0805_2012Metric_Pad1.15x1.40mm_HandSolder" V 6930 2600 50  0001 C CNN
 F 3 "~" H 7000 2600 50  0001 C CNN
