File: board/vfo.sch (KiCad schematic (older format))
At the start: 20 parts, among them J1 CVIN, J2 SAW, J3 TRI, J4 Conn_02x05_Odd_Even, J5 Conn_01x06, U1 TL072, U2 AS3340

Commit message: Use correct resistor value
Parts:
- R6: value 820R -> 620R
Changed lines of the file:
@@
 P 9800 2600
 F 0 "R6" H 9650 2600 50  0000 L CNN
-F 1 "820R" V 9800 2500 50  0000 L CNN
+F 1 "620R" V 9800 2500 50  0000 L CNN
 F 2 "Resistor_SMD:R_0805_2012Metric_Pad1.15x1.40mm_HandSolder" V 9730 2600 50  0001 C CNN
 F 3 "~" H 9800 2600 50  0001 C CNN

Commit message: Add missing 100K resistor
Parts:
- added R9: 100K, Resistor_SMD:R_0805_2012Metric_Pad1.15x1.40mm_HandSolder, symbol Device:R
- RV2: MPN ‎3314J-1-103E -> 3314J-1-103E
- U1: MPN ‎TL072CDR -> TL072CDR
Changed lines of the file:
@@
 F 3 "~" H 6750 1100 50  0001 C CNN
 F 4 "Bourns" H 0   0   50  0001 C CNN "MFR"
-F 5 "‎3314J-1-103E" H 0   0   50  0001 C CNN "MPN"
+F 5 "3314J-1-103E" H 0   0   50  0001 C CNN "MPN"
 F 6 "-" H 0   0   50  0001 C CNN "SPR"
 F 7 "-" H 0   0   50  0001 C CNN "SPN"
@@
 F 3 "http://www.ti.com/lit/ds/symlink/tl071.pdf" H 4400 1400 50  0001 C CNN
 F 4 "-" H 0   0   50  0001 C CNN "MFR"
-F 5 " ‎TL072CDR" H 0   0   50  0001 C CNN "MPN"
+F 5 "TL072CDR" H 0   0   50  0001 C CNN "MPN"
 F 6 "-" H 0   0   50  0001 C CNN "SPR"
 F 7 "-" H 0   0   50  0001 C CNN "SPN"
@@
 F 3 "http://www.ti.com/lit/ds/symlink/tl071.pdf" H 4400 2150 50  0001 C CNN
 F 4 "-" H 0   0   50  0001 C CNN "MFR"
-F 5 " ‎TL072CDR" H 0   0   50  0001 C CNN "MPN"
+F 5 "TL072CDR" H 0   0   50  0001 C CNN "MPN"
 F 6 "-" H 0   0   50  0001 C CNN "SPR"
 F 7 "-" H 0   0   50  0001 C CNN "SPN"
@@
 L Device:R_POT RV1
 U 1 1 5B6D2DC3
-P 6700 2200
-F 0 "RV1" V 6600 2200 50  0000 C CNN
-F 1 "100K" V 6700 2200 50  0000 C CNN
-F 2 "Connector_PinHeader_2.54mm:PinHeader_1x03_P2.54mm_Vertical" H 6700 2200 50  0001 C CNN
-F 3 "~" H 6700 2200 50  0001 C CNN
-F 4 "-" H 0   0   50  0001 C CNN "MFR"
-F 5 "-" H 0   0   50  0001 C CNN "MPN"
-F 6 "-" H 0   0   50  0001 C CNN "SPR"
-F 7 "-" H 0   0   50  0001 C CNN "SPN"
-F 8 "-" H 0   0   50  0001 C CNN "SPURL"
-	1    6700 2200
+P 6700 1900
+F 0 "RV1" V 6600 1900 50  0000 C CNN
+F 1 "100K" V 6700 1900 50  0000 C CNN
+F 2 "Connector_PinHeader_2.54mm:PinHeader_1x03_P2.54mm_Vertical" H 6700 1900 50  0001 C CNN
+F 3 "~" H 6700 1900 50  0001 C CNN
+F 4 "-" H 0   -300 50  0001 C CNN "MFR"
+F 5 "-" H 0   -300 50  0001 C CNN "MPN"
+F 6 "-" H 0   -300 50  0001 C CNN "SPR"
+F 7 "-" H 0   -300 50  0001 C CNN "SPN"
+F 8 "-" H 0   -300 50  0001 C CNN "SPURL"
+	1    6700 1900
 	0    1    1    0
 $EndComp
@@
 L power:+12V #PWR0120
 U 1 1 5B70A098
-P 6850 2200
-F 0 "#PWR0120" H 6850 2050 50  0001 C CNN
-F 1 "+12V" V 6865 2328 50  0000 L CNN
-F 2 "" H 6850 2200 50  0001 C CNN
-F 3 "" H 6850 2200 50  0001 C CNN
-	1    6850 2200
+P 6850 1900
+F 0 "#PWR0120" H 6850 1750 50  0001 C CNN
+F 1 "+12V" V 6865 2028 50  0000 L CNN
+F 2 "" H 6850 1900 50  0001 C CNN
+F 3 "" H 6850 1900 50  0001 C CNN
+	1    6850 1900
 	0    1    1    0
 $EndComp
@@
 	6350 2000 6350 2300
 Wire Wire Line
-	6350 2600 6700 2600
-Wire Wire Line
-	6700 2350 6700 2400
-Wire Wire Line
-	6700 2600 6850 2600
-Wire Wire Line
-	6550 2200 6550 2400
-Wire Wire Line
-	6550 2400 6700 2400
-Wire Wire Line
-	6700 2400 6700 2600
+	6700 2050 6700 2100
+Wire Wire Line
+	6550 1900 6550 2100
+Wire Wire Line
+	6550 2100 6700 2100
+Wire Wire Line
+	6700 2100 6700 2300
 Wire Notes Line
 	7950 500  7950 3250
@@
 Connection ~ 10500 3000
 Connection ~ 6350 2600
+Connection ~ 6700 2100
+Connection ~ 9800 2350
+Wire Wire Line
+	6350 2600 6700 2600
+$Comp
+L Device:R R9
+U 1 1 5B8F6E6E
+P 6700 2450
+F 0 "R9" H 6550 2500 50  0000 L CNN
+F 1 "100K" V 6700 2350 50  0000 L CNN
+F 2 "Resistor_SMD:R_0805_2012Metric_Pad1.15x1.40mm_HandSolder" V 6630 2450 50  0001 C CNN
+F 3 "~" H 6700 2450 50  0001 C CNN
+	1    6700 2450
+	1    0    0    -1
+$EndComp
 Connection ~ 6700 2600
-Connection ~ 6700 2400
-Connection ~ 9800 2350
+Wire Wire Line
+	6700 2600 6850 2600
 $EndSCHEMATC

Commit message: Break into two boards
Parts:
- removed J1: CVIN, Connector_PinHeader_2.54mm:PinHeader_1x02_P2.54mm_Vertical, symbol Connector_Generic:Conn_01x02
- removed J2: SAW, Connector_PinHeader_2.54mm:PinHeader_1x02_P2.54mm_Vertical, symbol Connector_Generic:Conn_01x02
- removed J3: TRI, Connector_PinHeader_2.54mm:PinHeader_1x02_P2.54mm_Vertical, symbol Connector_Generic:Conn_01x02
- added J1: CVIN, Connector_Audio:Jack_3.5mm_QingPu_WQP-PJ398SM_Vertical_CircularHoles, symbol Connector:AudioJack2_Ground_Switch
- added J2: SAW, Connector_Audio:Jack_3.5mm_QingPu_WQP-PJ398SM_Vertical_CircularHoles, symbol Connector:AudioJack2_Ground_Switch
- added J3: TRI, Connector_Audio:Jack_3.5mm_QingPu_WQP-PJ398SM_Vertical_CircularHoles, symbol Connector:AudioJack2_Ground_Switch
- added J6: Daughter_top, Connector_PinSocket_2.54mm:PinSocket_1x03_P2.54mm_Vertical, symbol Connector:Conn_01x03_Female
- added J7: Mother_top, Connector_PinHeader_2.54mm:PinHeader_1x03_P2.54mm_Vertical, symbol Connector:Conn_01x03_Male
- added J8: Daughter_bottom, Connector_PinSocket_2.54mm:PinSocket_1x03_P2.54mm_Vertical, symbol Connector:Conn_01x03_Female
- added J9: Mother_bottom, Connector_PinHeader_2.54mm:PinHeader_1x03_P2.54mm_Vertical, symbol Connector:Conn_01x03_Male
- RV1: footprint Connector_PinHeader_2.54mm:PinHeader_1x03_P2.54mm_Vertical -> Potentiometer_THT:Potentiometer_Alps_RK09L_Single_Vertical
Connections:
- net labels added: CV_IN, D_12V, D_CV_IN, D_GND, D_SAW_OUT, D_TRI_OUT, D_TUNE_POT, TUNE_POT
- net labels removed: CVIN
- wire segments 55 -> 72
- no-connect marks 0 -> 3
Other:
- note added: "Front Panel Board"

Commit message: Add protection diodes
Parts:
- added D1, D2: DIODE, Diode_SMD:D_0805_2012Metric_Pad1.15x1.40mm_HandSolder, symbol pspice:DIODE
Connections:
- net labels added: -12V_IN, 12V_IN
- wire segments 72 -> 78
Changed lines of the file:
@@
-$EndComp
-$Comp
-L power:+12V #PWR0130
-U 1 1 5B6FAF85
-P 10350 3600
-F 0 "#PWR0130" H 10350 3450 50  0001 C CNN
-F 1 "+12V" V 10350 3750 50  0000 L CNN
-F 2 "" H 10350 3600 50  0001 C CNN
-F 3 "" H 10350 3600 50  0001 C CNN
-	1    10350 3600
-	0    1    1    0
 $EndComp
 $Comp
 L power:-12V #PWR0131
 U 1 1 5B6FAF8B
-P 10350 4000
-F 0 "#PWR0131" H 10350 4100 50  0001 C CNN
-F 1 "-12V" V 10350 4150 50  0000 L CNN
-F 2 "" H 10350 4000 50  0001 C CNN
-F 3 "" H 10350 4000 50  0001 C CNN
-	1    10350 4000
+P 6850 3950
+F 0 "#PWR0131" H 6850 4050 50  0001 C CNN
+F 1 "-12V" V 6850 4100 50  0000 L CNN
+F 2 "" H 6850 3950 50  0001 C CNN
+F 3 "" H 6850 3950 50  0001 C CNN
+	1    6850 3950
 	0    1    1    0
 $EndComp
@@
 L power:+12V #PWR0135
 U 1 1 5B6FC19D
-P 9850 3600
-F 0 "#PWR0135" H 9850 3450 50  0001 C CNN
-F 1 "+12V" V 9850 3750 50  0000 L CNN
-F 2 "" H 9850 3600 50  0001 C CNN
-F 3 "" H 9850 3600 50  0001 C CNN
-	1    9850 3600
-	0    -1   -1   0
-$EndComp
-$Comp
-L power:-12V #PWR0136
-U 1 1 5B6FC1A3
-P 9850 4000
-F 0 "#PWR0136" H 9850 4100 50  0001 C CNN
-F 1 "-12V" V 9850 4150 50  0000 L CNN
-F 2 "" H 9850 4000 50  0001 C CNN
-F 3 "" H 9850 4000 50  0001 C CNN
-	1    9850 4000
-	0    -1   -1   0
+P 6850 3650
+F 0 "#PWR0135" H 6850 3500 50  0001 C CNN
+F 1 "+12V" V 6850 3800 50  0000 L CNN
+F 2 "" H 6850 3650 50  0001 C CNN
+F 3 "" H 6850 3650 50  0001 C CNN
+	1    6850 3650
+	0    1    1    0
 $EndComp
 $Comp
@@
 	1    0    0    -1
 $EndComp
+$Comp
+L pspice:DIODE D1
+U 1 1 5BA0E791
+P 6650 3650
+F 0 "D1" H 6650 3915 50  0000 C CNN
+F 1 "DIODE" H 6650 3824 50  0000 C CNN
+F 2 "Diode_SMD:D_0805_2012Metric_Pad1.15x1.40mm_HandSolder" H 6650 3650 50  0001 C CNN
+F 3 "" H 6650 3650 50  0001 C CNN
+	1    6650 3650
+	1    0    0    -1
+$EndComp
+$Comp
+L pspice:DIODE D2
+U 1 1 5BA0E85B
+P 6650 3950
+F 0 "D2" H 6650 4215 50  0000 C CNN
+F 1 "DIODE" H 6650 4124 50  0000 C CNN
+F 2 "Diode_SMD:D_0805_2012Metric_Pad1.15x1.40mm_HandSolder" H 6650 3950 50  0001 C CNN
+F 3 "" H 6650 3950 50  0001 C CNN
+	1    6650 3950
+	-1   0    0    1
+$EndComp
+Wire Wire Line
+	9850 3600 9550 3600
+Text Label 9550 3600 0    50   ~ 0
+12V_IN
+Wire Wire Line
+	10350 3600 10700 3600
+Text Label 10700 3600 2    50   ~ 0
+12V_IN
+Wire Wire Line
+	6450 3650 6100 3650
+Text Label 6100 3650 0    50   ~ 0
+12V_IN
+Wire Wire Line
+	6450 3950 6050 3950
+Text Label 6050 3950 0    50   ~ 0
+-12V_IN
+Wire Wire Line
+	9850 4000 9500 4000
+Text Label 9500 4000 0    50   ~ 0
+-12V_IN
+Wire Wire Line
+	10350 4000 10700 4000
+Text Label 10700 4000 2    50   ~ 0
+-12V_IN
+Wire Notes Line
+	7500 4300 5750 4300
+Wire Notes Line
+	5750 4300 5750 3250
 $EndSCHEMATC
